File: hardware/kicad/base_station.kicad_sch (KiCad schematic)
At the start: 4 parts, among them U1 Arduino UNO Q (STM32U585 side), U2 SmartElex KX134-1211 (acceler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, U3 INMP441 (I2S microphone), U4 WS2812B x8 status ring

Commit message: schematics: name controller pins the way the boards name them
The three KiCad schematics labelled every controller pin by its MCU function
or STM32 port -- SCK, MISO, I2S_CLK, LED_DIN, PB0 -- which is not what any of
these boards is silkscreened with and not what you plug a wire into. Someone
holding an UNO Q and the schematic had no way to find "I2S_CLK".

Pins now carry the board's own header labels: D13/D12/D11/D8/D9/SCL/D10/A4/D3
on the UNO Q, D0-D10 on the XIAO, D2-D8 on the Uno under the CNC shield. The
signal's role moves into the net label, where it was already half-living
(SPI_SCK_D13, MIC_SD_A4), so each sensor stub still says both what the line
carries and which header pin it lands on. Sensor and driver symbols keep
their datasheet names -- those breakouts really are marked SCK/SDO/STEP.

Two labels were also just wrong, not merely inconvenient: the ring's DIN read
LED_DIN_PB0 when PB0 is header pin D3, and the mic's three lines read
PB10/PB9/PC1 with no header pin at all -- they are SCL, D10 and A4. Mapping is
the board's own gpio-map (arduino_r3_connector.dtsi) for the UNO Q and
board_pins.h for the XIAO; the mic's bit clock is genuinely the odd one out,
since PB10 comes out as the dedicated SCL pin rather than a D-number.

Appendix B.1's table gains the same treatment, and the report PNGs are
re-cropped to the drawing rather than the sheet -- they were carrying about
half a page of blank paper each, which shrank the schematic on the page. The
crop is now derived in the README instead of living in shell history.

Co-Authored-By: Claude Opus 5 <noreply@anthropic.com>
Connections:
- net LED_DIN_PB0 renamed LED_DIN_D3
- net MIC_SCK_PB10 renamed MIC_SCK_SCL
- net MIC_SD_PC1 renamed MIC_SD_A4
- net MIC_WS_PB9 renamed MIC_WS_D10
Other:
- note added: "Report ref: Chapter 2.3 / Appendix B.1. UNO Q pins are named by its own header labels (D3, D13, A4, SCL) -- not by STM32 port."
- note removed: "Report ref: Chapter 2.3 / Appendix B.1. Net labels carry the header pin used on the UNO Q main header."
Changed lines of the file:
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@@
 		(effects (font (size 1.27 1.27)) (justify left))
 	)
-	(label "MIC_SCK_PB10"
+	(label "MIC_SCK_SCL"
 		(at 94.29 96.825 0)
 		(effects (font (size 1.27 1.27)) (justify left))
 	)
-	(label "MIC_WS_PB9"
+	(label "MIC_WS_D10"
 		(at 94.29 103.175 0)
 		(effects (font (size 1.27 1.27)) (justify left))
 	)
-	(label "MIC_SD_PC1"
+	(label "MIC_SD_A4"
 		(at 94.29 109.525 0)
 		(effects (font (size 1.27 1.27)) (justify left))
 	)
-	(label "LED_DIN_PB0"
+	(label "LED_DIN_D3"
 		(at 94.29 115.875 0)
 		(effects (font (size 1.27 1.27)) (justify left))
@@
 		(effects (font (size 1.27 1.27)) (justify right))
 	)
-	(label "MIC_SCK_PB10"
+	(label "MIC_SCK_SCL"
 		(at 144.60000000000002 109.125 0)
 		(effects (font (size 1.27 1.27)) (justify right))
 	)
-	(label "MIC_WS_PB9"
+	(label "MIC_WS_D10"
 		(at 144.60000000000002 115.475 0)
 		(effects (font (size 1.27 1.27)) (justify right))
 	)
-	(label "MIC_SD_PC1"
+	(label "MIC_SD_A4"
 		(at 144.60000000000002 121.825 0)
 		(effects (font (size 1.27 1.27)) (justify right))
 	)
-	(label "LED_DIN_PB0"
+	(label "LED_DIN_D3"
 		(at 144.60000000000002 163.65 0)
 		(effects (font (size 1.27 1.27)) (justify right))
@@
 		(effects (font (size 1.8 1.8)) (justify left))
 	)
-	(text "Report ref: Chapter 2.3 / Appendix B.1. Net labels carry the header pin used on the UNO Q main header."
+	(text "Report ref: Chapter 2.3 / Appendix B.1. UNO Q pins are named by its own header labels (D3, D13, A4, SCL) -- not by STM32 port."
 		(exclude_from_sim no)
 		(at 20 38 0)
@@
 		(instances
 			(project "epm"
-				(path "/9925249e-0a56-43fc-ae23-61604831cde2"
+				(path "/ee415933-6b43-4ace-8980-e1947a4ed4ca"
 					(reference "U1")
 					(unit 1)
@@
 		(on_board yes)
 		(dnp no)
-		(property "Reference" "#PWReeaf"
+		(property "Reference" "#PWRef9d"
 			(at 94.29 118.41499999999999 0)
 			(effects (font (size 1.27 1.27)) (hide yes))
@@
 		(instances
 			(project "epm"
-				(path "/9925249e-0a56-43fc-ae23-61604831cde2"
-					(reference "#PWReeaf")
+				(path "/ee415933-6b43-4ace-8980-e1947a4ed4ca"
+					(reference "#PWRef9d")
 					(unit 1)
 				)
@@
 		(on_board yes)
 		(dnp no)
-		(property "Reference" "#PWR903d"
+		(property "Reference" "#PWRf00f"
 			(at 94.29 124.76499999999999 0)
 			(effects (font (size 1.27 1.27)) (hide yes))
@@
 		(instances
 			(project "epm"
-				(path "/9925249e-0a56-43fc-ae23-61604831cde2"
-					(reference "#PWR903d")
+				(path "/ee415933-6b43-4ace-8980-e1947a4ed4ca"
+					(reference "#PWRf00f")
 					(unit 1)
 				)
@@
 		(on_board yes)
 		(dnp no)
-		(property "Reference" "#PWRe9c2"
+		(property "Reference" "#PWRf8a1"
 			(at 94.29 131.115 0)
 			(effects (font (size 1.27 1.27)) (hide yes))
@@
 		(instances
 			(project "epm"
-				(path "/9925249e-0a56-43fc-ae23-61604831cde2"
-					(reference "#PWRe9c2")
+				(path "/ee415933-6b43-4ace-8980-e1947a4ed4ca"
+					(reference "#PWRf8a1")
 					(unit 1)
 				)
@@
 		(instances
 			(project "epm"
-				(path "/9925249e-0a56-43fc-ae23-61604831cde2"
+				(path "/ee415933-6b43-4ace-8980-e1947a4ed4ca"
 					(reference "U2")
 					(unit 1)
@@
 		(on_board yes)
 		(dnp no)
-		(property "Reference" "#PWR3519"
+		(property "Reference" "#PWR6d2e"
 			(at 143.32999999999998 78.89 0)
 			(effects (font (size 1.27 1.27)) (hide yes))
@@
 		(instances
 			(project "epm"
-				(path "/9925249e-0a56-43fc-ae23-61604831cde2"
-					(reference "#PWR3519")
+				(path "/ee415933-6b43-4ace-8980-e1947a4ed4ca"
+					(reference "#PWR6d2e")
 					(unit 1)
 				)
@@
 		(on_board yes)
 		(dnp no)
-		(property "Reference" "#PWRe792"
+		(property "Reference" "#PWR9204"
 			(at 143.32999999999998 85.24 0)
 			(effects (font (size 1.27 1.27)) (hide yes))
@@
 		(instances
 			(project "epm"
-				(path "/9925249e-0a56-43fc-ae23-61604831cde2"
-					(reference "#PWRe792")
+				(path "/ee415933-6b43-4ace-8980-e1947a4ed4ca"
+					(reference "#PWR9204")
 					(unit 1)
 				)
@@
 		(instances
 			(project "epm"
-				(path "/9925249e-0a56-43fc-ae23-61604831cde2"
+				(path "/ee415933-6b43-4ace-8980-e1947a4ed4ca"
 					(reference "U3")
 					(unit 1)
@@
 		(on_board yes)
 		(dnp no)
-		(property "Reference" "#PWR994a"
+		(property "Reference" "#PWR46a5"
 			(at 144.60000000000002 124.36500000000001 0)
 			(effects (font (size 1.27 1.27)) (hide yes))
@@
 		(instances
 			(project "epm"
-				(path "/9925249e-0a56-43fc-ae23-61604831cde2"
-					(reference "#PWR994a")
+				(path "/ee415933-6b43-4ace-8980-e1947a4ed4ca"
+					(reference "#PWR46a5")
 					(unit 1)
 				)
@@
 		(on_board yes)
 		(dnp no)
-		(property "Reference" "#PWR1edc"
+		(property "Reference" "#PWR4ef3"
 			(at 144.60000000000002 130.715 0)
 			(effects (font (size 1.27 1.27)) (hide yes))
@@
 		(instances
 			(project "epm"
-				(path "/9925249e-0a56-43fc-ae23-61604831cde2"
-					(reference "#PWR1edc")
+				(path "/ee415933-6b43-4ace-8980-e1947a4ed4ca"
+					(reference "#PWR4ef3")
 					(unit 1)
 				)
@@
 		(on_board yes)
 		(dnp no)
-		(property "Reference" "#PWRfa82"
+		(property "Reference" "#PWR79f1"
 			(at 144.60000000000002 137.065 0)
 			(effects (font (size 1.27 1.27)) (hide yes))
@@
 		(instances
 			(project "epm"
-				(path "/9925249e-0a56-43fc-ae23-61604831cde2"
-					(reference "#PWRfa82")
+				(path "/ee415933-6b43-4ace-8980-e1947a4ed4ca"
+					(reference "#PWR79f1")
 					(unit 1)
 				)
@@
 		(instances
 			(project "epm"
-				(path "/9925249e-0a56-43fc-ae23-61604831cde2"
+				(path "/ee415933-6b43-4ace-8980-e1947a4ed4ca"
 					(reference "U4")
 					(unit 1)
@@
 		(on_board yes)
 		(dnp no)
-		(property "Reference" "#PWR0e21"
+		(property "Reference" "#PWR2bbc"
 			(at 144.60000000000002 166.19 0)
 			(effects (font (size 1.27 1.27)) (hide yes))
@@
 		(instances
 			(project "epm"
-				(path "/9925249e-0a56-43fc-ae23-61604831cde2"
-					(reference "#PWR0e21")
+				(path "/ee415933-6b43-4ace-8980-e1947a4ed4ca"
+					(reference "#PWR2bbc")
 					(unit 1)
 				)
@@
 		(on_board yes)
 		(dnp no)
-		(property "Reference" "#PWRcc59"
+		(property "Reference" "#PWRe341"
 			(at 144.60000000000002 172.54 0)
 			(effects (font (size 1.27 1.27)) (hide yes))
@@
 		(instances
 			(project "epm"
-				(path "/9925249e-0a56-43fc-ae23-61604831cde2"
-					(reference "#PWRcc59")
-					(unit 1)
-				)
+				(path "/ee415933-6b43-4ace-8980-e1947a4ed4ca"
+					(reference "#PWRe341")
+					(unit 1)
+				)

Commit message: schematics: drop redundant pin-number suffix from net labels
The symbol pin already shows the pin number (D8, A4, SCL, ...), so
repeating it in the net label (SPI_SCK_D8) was noise. Net labels now
carry only the signal role (SPI_SCK, MIC_SD, ENABLE, ...).

Co-Authored-By: Claude Sonnet 5 <noreply@anthropic.com>
Connections:
- net ACC_CS_D8 renamed ACC_CS
- net ACC_INT_D9 renamed ACC_INT
- net LED_DIN_D3 renamed LED_DIN
- net MIC_SCK_SCL renamed MIC_SCK
- net MIC_SD_A4 renamed MIC_SD
- net MIC_WS_D10 renamed MIC_WS
- net SPI_MISO_D12 renamed SPI_MISO
- net SPI_MOSI_D11 renamed SPI_MOSI
- net SPI_SCK_D13 renamed SPI_SCK
Changed lines of the file:
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@@
 		(stroke (width 0) (type default))
 	)
-	(label "SPI_SCK_D13"
+	(label "SPI_SCK"
 		(at 94.29 65.075 0)
 		(effects (font (size 1.27 1.27)) (justify left))
 	)
-	(label "SPI_MISO_D12"
+	(label "SPI_MISO"
 		(at 94.29 71.425 0)
 		(effects (font (size 1.27 1.27)) (justify left))
 	)
-	(label "SPI_MOSI_D11"
+	(label "SPI_MOSI"
 		(at 94.29 77.775 0)
 		(effects (font (size 1.27 1.27)) (justify left))
 	)
-	(label "ACC_CS_D8"
+	(label "ACC_CS"
 		(at 94.29 84.125 0)
 		(effects (font (size 1.27 1.27)) (justify left))
 	)
-	(label "ACC_INT_D9"
+	(label "ACC_INT"
 		(at 94.29 90.475 0)
 		(effects (font (size 1.27 1.27)) (justify left))
 	)
-	(label "MIC_SCK_SCL"
+	(label "MIC_SCK"
 		(at 94.29 96.825 0)
 		(effects (font (size 1.27 1.27)) (justify left))
 	)
-	(label "MIC_WS_D10"
+	(label "MIC_WS"
 		(at 94.29 103.175 0)
 		(effects (font (size 1.27 1.27)) (justify left))
 	)
-	(label "MIC_SD_A4"
+	(label "MIC_SD"
 		(at 94.29 109.525 0)
 		(effects (font (size 1.27 1.27)) (justify left))
 	)
-	(label "LED_DIN_D3"
+	(label "LED_DIN"
 		(at 94.29 115.875 0)
 		(effects (font (size 1.27 1.27)) (justify left))
 	)
-	(label "SPI_SCK_D13"
+	(label "SPI_SCK"
 		(at 143.32999999999998 50.95 0)
 		(effects (font (size 1.27 1.27)) (justify right))
 	)
-	(label "SPI_MISO_D12"
+	(label "SPI_MISO"
 		(at 143.32999999999998 57.3 0)
 		(effects (font (size 1.27 1.27)) (justify right))
 	)
-	(label "SPI_MOSI_D11"
+	(label "SPI_MOSI"
 		(at 143.32999999999998 63.65 0)
 		(effects (font (size 1.27 1.27)) (justify right))
 	)
-	(label "ACC_CS_D8"
+	(label "ACC_CS"
 		(at 143.32999999999998 70.0 0)
 		(effects (font (size 1.27 1.27)) (justify right))
 	)
-	(label "ACC_INT_D9"
+	(label "ACC_INT"
 		(at 143.32999999999998 76.35 0)
 		(effects (font (size 1.27 1.27)) (justify right))
 	)
-	(label "MIC_SCK_SCL"
+	(label "MIC_SCK"
 		(at 144.60000000000002 109.125 0)
 		(effects (font (size 1.27 1.27)) (justify right))
 	)
-	(label "MIC_WS_D10"
+	(label "MIC_WS"
 		(at 144.60000000000002 115.475 0)
 		(effects (font (size 1.27 1.27)) (justify right))
 	)
-	(label "MIC_SD_A4"
+	(label "MIC_SD"
 		(at 144.60000000000002 121.825 0)
 		(effects (font (size 1.27 1.27)) (justify right))
 	)
-	(label "LED_DIN_D3"
+	(label "LED_DIN"
 		(at 144.60000000000002 163.65 0)
 		(effects (font (size 1.27 1.27)) (justify right))
@@
 		(instances
 			(project "epm"
-				(path "/ee415933-6b43-4ace-8980-e1947a4ed4ca"
+				(path "/971b503a-3d7a-446b-ac74-d56031e86485"
 					(reference "U1")
 					(unit 1)
@@
 		(on_board yes)
 		(dnp no)
-		(property "Reference" "#PWRef9d"
+		(property "Reference" "#PWRad90"
 			(at 94.29 118.41499999999999 0)
 			(effects (font (size 1.27 1.27)) (hide yes))
@@
 		(instances
 			(project "epm"
-				(path "/ee415933-6b43-4ace-8980-e1947a4ed4ca"
-					(reference "#PWRef9d")
+				(path "/971b503a-3d7a-446b-ac74-d56031e86485"
+					(reference "#PWRad90")
 					(unit 1)
 				)
@@
 		(on_board yes)
 		(dnp no)
-		(property "Reference" "#PWRf00f"
+		(property "Reference" "#PWR800b"
 			(at 94.29 124.76499999999999 0)
 			(effects (font (size 1.27 1.27)) (hide yes))
@@
 		(instances
 			(project "epm"
-				(path "/ee415933-6b43-4ace-8980-e1947a4ed4ca"
-					(reference "#PWRf00f")
+				(path "/971b503a-3d7a-446b-ac74-d56031e86485"
+					(reference "#PWR800b")
 					(unit 1)
 				)
@@
 		(on_board yes)
 		(dnp no)
-		(property "Reference" "#PWRf8a1"
+		(property "Reference" "#PWRd112"
 			(at 94.29 131.115 0)
 			(effects (font (size 1.27 1.27)) (hide yes))
@@
 		(instances
 			(project "epm"
-				(path "/ee415933-6b43-4ace-8980-e1947a4ed4ca"
-					(reference "#PWRf8a1")
+				(path "/971b503a-3d7a-446b-ac74-d56031e86485"
+					(reference "#PWRd112")
 					(unit 1)
 				)
@@
 		(instances
 			(project "epm"
-				(path "/ee415933-6b43-4ace-8980-e1947a4ed4ca"
+				(path "/971b503a-3d7a-446b-ac74-d56031e86485"
 					(reference "U2")
 					(unit 1)
@@
 		(on_board yes)
 		(dnp no)
-		(property "Reference" "#PWR6d2e"
+		(property "Reference" "#PWR2f59"
 			(at 143.32999999999998 78.89 0)
 			(effects (font (size 1.27 1.27)) (hide yes))
@@
 		(instances
 			(project "epm"
-				(path "/ee415933-6b43-4ace-8980-e1947a4ed4ca"
-					(reference "#PWR6d2e")
+				(path "/971b503a-3d7a-446b-ac74-d56031e86485"
+					(reference "#PWR2f59")
 					(unit 1)
 				)
@@
 		(on_board yes)
 		(dnp no)
-		(property "Reference" "#PWR9204"
+		(property "Reference" "#PWR85c2"
 			(at 143.32999999999998 85.24 0)
 			(effects (font (size 1.27 1.27)) (hide yes))
@@
 		(instances
 			(project "epm"
-				(path "/ee415933-6b43-4ace-8980-e1947a4ed4ca"
-					(reference "#PWR9204")
+				(path "/971b503a-3d7a-446b-ac74-d56031e86485"
+					(reference "#PWR85c2")
 					(unit 1)
 				)
@@
 		(instances
 			(project "epm"
-				(path "/ee415933-6b43-4ace-8980-e1947a4ed4ca"
+				(path "/971b503a-3d7a-446b-ac74-d56031e86485"
 					(reference "U3")
 					(unit 1)
@@
 		(on_board yes)
 		(dnp no)
-		(property "Reference" "#PWR46a5"
+		(property "Reference" "#PWRa40e"
 			(at 144.60000000000002 124.36500000000001 0)
 			(effects (font (size 1.27 1.27)) (hide yes))
@@
 		(instances
 			(project "epm"
-				(path "/ee415933-6b43-4ace-8980-e1947a4ed4ca"
-					(reference "#PWR46a5")
+				(path "/971b503a-3d7a-446b-ac74-d56031e86485"
+					(reference "#PWRa40e")
 					(unit 1)
 				)
@@
 		(on_board yes)
 		(dnp no)
-		(property "Reference" "#PWR4ef3"
+		(property "Reference" "#PWRb739"
 			(at 144.60000000000002 130.715 0)
 			(effects (font (size 1.27 1.27)) (hide yes))
@@
 		(instances
 			(project "epm"
-				(path "/ee415933-6b43-4ace-8980-e1947a4ed4ca"
-					(reference "#PWR4ef3")
+				(path "/971b503a-3d7a-446b-ac74-d56031e86485"
+					(reference "#PWRb739")
 					(unit 1)
 				)
@@
 		(on_board yes)
 		(dnp no)
-		(property "Reference" "#PWR79f1"
+		(property "Reference" "#PWR3135"
 			(at 144.60000000000002 137.065 0)
 			(effects (font (size 1.27 1.27)) (hide yes))
@@
 		(instances
 			(project "epm"
-				(path "/ee415933-6b43-4ace-8980-e1947a4ed4ca"
-					(reference "#PWR79f1")
+				(path "/971b503a-3d7a-446b-ac74-d56031e86485"
+					(reference "#PWR3135")
 					(unit 1)
 				)
@@
 		(instances
 			(project "epm"
-				(path "/ee415933-6b43-4ace-8980-e1947a4ed4ca"
+				(path "/971b503a-3d7a-446b-ac74-d56031e86485"
 					(reference "U4")
 					(unit 1)
@@
 		(on_board yes)
 		(dnp no)
-		(property "Reference" "#PWR2bbc"
+		(property "Reference" "#PWR873d"
 			(at 144.60000000000002 166.19 0)
 			(effects (font (size 1.27 1.27)) (hide yes))
@@
 		(instances
 			(project "epm"
-				(path "/ee415933-6b43-4ace-8980-e1947a4ed4ca"
-					(reference "#PWR2bbc")
+				(path "/971b503a-3d7a-446b-ac74-d56031e86485"
+					(reference "#PWR873d")
 					(unit 1)
 				)
@@
 		(on_board yes)
 		(dnp no)
-		(property "Reference" "#PWRe341"
+		(property "Reference" "#PWR9333"
 			(at 144.60000000000002 172.54 0)
 			(effects (font (size 1.27 1.27)) (hide yes))
@@
 		(instances
 			(project "epm"
-				(path "/ee415933-6b43-4ace-8980-e1947a4ed4ca"
-					(reference "#PWRe341")
-					(unit 1)
-				)
+				(path "/971b503a-3d7a-446b-ac74-d56031e86485"
+					(reference "#PWR9333")
+					(unit 1)
+				)
